File: Minisumo/Minisumo.sch (KiCad schematic (older format))
At the start: 103 parts, among them IC1 ATMEGA328P-A, P1 bateria, P2 PROGRAMATOR, P3 silnik2, P4 silnik1, U1 LM1117_5V, U10 KTIR0711S, U11 MMA7455L, U12 SFH7773, U13 74HC595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

Commit message: poprawa schematu
nieznaczna poprawa schematu 13
Parts:
- removed R?: 100, symbol R
- removed R?: 10k, symbol R
- removed U?: transoptor, warsztaty:KTIR0711S, symbol KTIR0711S
- U3: value TSOP4836 -> TSOP4838
Connections:
- net ACC_DRDY: now also IC1.13 ((PCINT1/OC1A)PB1)
- net KILL: now also IC1.2 ((PCINT20/XCK/T0)PD4)
- no-connect marks 9 -> 6
Other:
- moved on the sheet: P?
Changed lines of the file:
@@
 Text Label 4400 7100 2    60   ~ 0
 ACC_INT2
-NoConn ~ 10700 10600
 Text Notes 9200 9700 0    60   ~ 0
 AKCELELOMETR
@@
 P 5850 7500
 F 0 "U3" V 5850 7900 60  0000 C CNN
-F 1 "TSOP4836" V 5550 7750 60  0000 C CNN
+F 1 "TSOP4838" V 5550 7750 60  0000 C CNN
 F 2 "LEDs:LED-5MM-3" H 5850 7500 60  0001 C CNN
 F 3 "" H 5850 7500 60  0000 C CNN
@@
 	0    -1   -1   0
 $EndComp
-NoConn ~ 4400 7500
 Text Label 4450 7400 2    60   ~ 0
 KTIR_PWM
@@
 Wire Wire Line
 	9900 7200 10450 7200
-NoConn ~ 4400 5600
-$Comp
-L KTIR0711S U?
-U 1 1 5644A79F
-P 6800 9750
-F 0 "U?" H 6600 9950 50  0000 L CNN
-F 1 "transoptor" H 6800 9950 50  0000 L CNN
-F 2 "warsztaty:KTIR0711S" H 6600 9550 50  0001 L CIN
-F 3 "" H 6800 9750 50  0000 L CNN
-	1    6800 9750
-	1    0    0    -1
-$EndComp
-$Comp
-L R R?
-U 1 1 5644D254
-P 6350 9650
-F 0 "R?" V 6430 9650 50  0000 C CNN
-F 1 "100" V 6350 9650 50  0000 C CNN
-F 2 "" V 6280 9650 30  0000 C CNN
-F 3 "" H 6350 9650 30  0000 C CNN
-	1    6350 9650
-	0    1    1    0
-$EndComp
-$Comp
-L GND #PWR?
-U 1 1 5644E89E
-P 6500 9850
-F 0 "#PWR?" H 6500 9600 50  0001 C CNN
-F 1 "GND" H 6500 9700 50  0000 C CNN
-F 2 "" H 6500 9850 60  0000 C CNN
-F 3 "" H 6500 9850 60  0000 C CNN
-	1    6500 9850
-	1    0    0    -1
-$EndComp
-$Comp
-L R R?
-U 1 1 5644E9E1
-P 7200 10100
-F 0 "R?" V 7280 10100 50  0000 C CNN
-F 1 "10k" V 7200 10100 50  0000 C CNN
-F 2 "" V 7130 10100 30  0000 C CNN
-F 3 "" H 7200 10100 30  0000 C CNN
-	1    7200 10100
-	-1   0    0    1
-$EndComp
-Wire Wire Line
-	7100 9850 7350 9850
-Wire Wire Line
-	7200 9850 7200 9950
-Wire Wire Line
-	6200 9350 6750 9350
-Text Label 6750 9350 2    60   ~ 0
-KILL
-$Comp
-L GND #PWR?
-U 1 1 564528FB
-P 7200 10250
-F 0 "#PWR?" H 7200 10000 50  0001 C CNN
-F 1 "GND" H 7200 10100 50  0000 C CNN
-F 2 "" H 7200 10250 60  0000 C CNN
-F 3 "" H 7200 10250 60  0000 C CNN
-	1    7200 10250
-	1    0    0    -1
-$EndComp
-Connection ~ 7200 9850
-Text Label 7350 9850 2    60   ~ 0
-VDD
-Wire Wire Line
-	7100 9650 7200 9650
-Wire Wire Line
-	7200 9650 7200 9350
-$Comp
-L +5V #PWR?
-U 1 1 564568E2
-P 7200 9350
-F 0 "#PWR?" H 7200 9200 50  0001 C CNN
-F 1 "+5V" H 7200 9490 50  0000 C CNN
-F 2 "" H 7200 9350 60  0000 C CNN
-F 3 "" H 7200 9350 60  0000 C CNN
-	1    7200 9350
-	1    0    0    -1
-$EndComp
 Wire Wire Line
 	12400 1250 12200 1250
@@
 VDD
 Wire Wire Line
-	6200 9650 6200 9350
-Wire Wire Line
 	12350 4100 12150 4100
 Text Label 12150 4100 0    60   ~ 0
 VDD
-Wire Notes Line
-	5250 10550 7550 10550
-Wire Notes Line
-	7550 9100 7550 10550
-Wire Notes Line
-	5250 9100 7550 9100
 $Comp
 L CONN_01X04 P?
 U 1 1 56461B59
-P 5650 9550
-F 0 "P?" H 5650 9800 50  0000 C CNN
-F 1 "CONN_01X04" V 5750 9550 50  0000 C CNN
-F 2 "" H 5650 9550 60  0000 C CNN
-F 3 "" H 5650 9550 60  0000 C CNN
-	1    5650 9550
+P 7150 4800
+F 0 "P?" H 7150 5050 50  0000 C CNN
+F 1 "CONN_01X04" V 7250 4800 50  0000 C CNN
+F 2 "" H 7150 4800 60  0000 C CNN
+F 3 "" H 7150 4800 60  0000 C CNN
+	1    7150 4800
 	0    -1   -1   0
 $EndComp
@@
 L +5V #PWR?
 U 1 1 564621AA
-P 5500 9750
-F 0 "#PWR?" H 5500 9600 50  0001 C CNN
-F 1 "+5V" H 5500 9890 50  0000 C CNN
-F 2 "" H 5500 9750 60  0000 C CNN
-F 3 "" H 5500 9750 60  0000 C CNN
-	1    5500 9750
+P 7000 5000
+F 0 "#PWR?" H 7000 4850 50  0001 C CNN
+F 1 "+5V" H 7000 5140 50  0000 C CNN
+F 2 "" H 7000 5000 60  0000 C CNN
+F 3 "" H 7000 5000 60  0000 C CNN
+	1    7000 5000
 	-1   0    0    1
 $EndComp
@@
 L GND #PWR?
 U 1 1 56462292
-P 5600 9750
-F 0 "#PWR?" H 5600 9500 50  0001 C CNN
-F 1 "GND" H 5600 9600 50  0000 C CNN
-F 2 "" H 5600 9750 60  0000 C CNN
-F 3 "" H 5600 9750 60  0000 C CNN
-	1    5600 9750
-	1    0    0    -1
-$EndComp
-Wire Wire Line
-	5700 9750 5700 10100
-Wire Wire Line
-	5800 9750 5800 10100
-Wire Wire Line
-	5800 10100 6000 10100
-Wire Wire Line
-	5700 10100 5400 10100
-Text Label 5400 10100 0    60   ~ 0
+P 7100 5000
+F 0 "#PWR?" H 7100 4750 50  0001 C CNN
+F 1 "GND" H 7100 4850 50  0000 C CNN
+F 2 "" H 7100 5000 60  0000 C CNN
+F 3 "" H 7100 5000 60  0000 C CNN
+	1    7100 5000
+	1    0    0    -1
+$EndComp
+Wire Wire Line
+	7200 5000 7200 5350
+Wire Wire Line
+	7300 5000 7300 5350
+Wire Wire Line
+	7300 5350 7500 5350
+Wire Wire Line
+	7200 5350 6900 5350
+Text Label 6900 5350 0    60   ~ 0
 START
-Text Label 6000 10100 2    60   ~ 0
+Text Label 7500 5350 2    60   ~ 0
 KILL
 Text Label 4400 7200 2    60   ~ 0
 START
 Wire Notes Line
-	5250 9100 5250 10550
-Text Notes 6000 9100 0    60   ~ 0
+	6750 4350 6750 5800
+Text Notes 6900 4350 0    60   ~ 0
 START MODULE\n
+Text Label 4400 7500 2    60   ~ 0
+KILL
+Text Label 4400 5600 2    60   ~ 0
+ACC_DRDY
+Wire Notes Line
+	7650 4350 7650 5800
+Wire Notes Line
+	7650 5800 6750 5800
+Wire Notes Line
+	6800 4350 7650 4350
 $EndSCHEMATC
