File: Minisumo uproszczony/Minisumo.sch (KiCad schematic (older format))
At the start: 100 parts, among them IC1 ATMEGA328P-A, P1 bateria, P2 PROGRAMATOR, P3 silnik2, P4 silnik1, U1 LM1117_5V, U10 KTIR0711S, U11 MMA7455L, U12 SFH7773, U13 74HC595, U14 TB6612, U15 TB6612, U16 SFH7773, U17 RGB_diode, U2 LM1117_3.3V, U3 TSOP4838, U4 SHARP_10-80, U5 SHARP_10-80, U6 LM339, U7 KTIR0711S, U8 KTIR0711S, U9 KTIR0711S, Y1 16mHz

Commit message: Bez komparatorow
uproszczono schemat
Parts:
- removed C22: 100nF, symbol C
- removed R10, R7, R8, R9: 47K, symbol R
- removed R15: 33K, symbol R
- removed R16, R17, R18, R19: 1K, symbol R
- removed U6: LM339, symbol LM339
- added R98, R99: 10K, symbol R
- added R?: 1k, Resistors_SMD:R_0805_HandSoldering, symbol R
- P3: renamed from P?; footprint (none) -> Pin_Headers:Pin_Header_Straight_1x04
- R3, R4, R5, R6: footprint (none) -> Resistors_SMD:R_0805_HandSoldering
- renumbered P3 to P4, P4 to P5
Connections:
- net labels removed: INT_KTIR_1, INT_KTIR_2, INT_KTIR_3, INT_KTIR_4, KTIR_PWM, POROWNANIE, VDD
- wire segments 388 -> 352
- no-connect marks 6 -> 7
Other:
- note removed: "WYKRYWANIE LINII\n"

Commit message: 3 Sharpy
dodano sharpa, dodano 2 attiny
Parts:
- added C?: 1uF, Capacitors_Elko_ThroughHole:Elko_vert_11x5mm_RM2, symbol CP
- added C?: 100nF, Capacitors_SMD:C_0805_HandSoldering, symbol C
- added IC? (x2): ATTINY13A-SS, SO8, symbol ATTINY13A-SS
- added P?: PROG_A1, symbol CONN_01X05
- added P?: PROG_A2, symbol CONN_01X05
- added R?: 6K8, Resistors_SMD:R_0805_HandSoldering, symbol R
- added R?: 22K, Resistors_SMD:R_0805_HandSoldering, symbol R
- added U?: SHARP_10-80, Pin_Headers:Pin_Header_Straight_1x03, symbol SHARP_10-80
- C1, C11, C12, C14, C15, C18, C19, C2, C20, C3, C4, C5, C8: footprint Capacitors_SMD:C_0805 -> Capacitors_SMD:C_0805_HandSoldering
- C24: renamed from C25; footprint Capacitors_SMD:C_0805 -> Capacitors_SMD:C_0805_HandSoldering
- C25: renamed from C26; footprint Capacitors_SMD:C_0805 -> Capacitors_SMD:C_0805_HandSoldering
- C28: renamed from C29; footprint Capacitors_SMD:C_0805 -> Capacitors_SMD:C_0805_HandSoldering
- C29: renamed from C30; footprint Capacitors_SMD:C_0805 -> Capacitors_SMD:C_0805_HandSoldering
- C30: renamed from C31; footprint Capacitors_SMD:C_0805 -> Capacitors_SMD:C_0805_HandSoldering
- C31: renamed from C32; footprint Capacitors_SMD:C_0805 -> Capacitors_SMD:C_0805_HandSoldering
- C32: renamed from C33; footprint Capacitors_SMD:C_0805 -> Capacitors_SMD:C_0805_HandSoldering
- C33: renamed from C34; footprint Capacitors_SMD:C_0805 -> Capacitors_SMD:C_0805_HandSoldering
- C34: renamed from C35; footprint Capacitors_SMD:C_0805 -> Capacitors_SMD:C_0805_HandSoldering
- C35: renamed from C36; footprint Capacitors_SMD:C_0805 -> Capacitors_SMD:C_0805_HandSoldering
- C37: renamed from C38; footprint Capacitors_SMD:C_0805 -> Capacitors_SMD:C_0805_HandSoldering
- C38: renamed from C39; footprint Capacitors_SMD:C_0805 -> Capacitors_SMD:C_0805_HandSoldering
- C39: renamed from C40; footprint Capacitors_SMD:C_0805 -> Capacitors_SMD:C_0805_HandSoldering
- C41: renamed from C42; footprint Capacitors_SMD:C_0805 -> Capacitors_SMD:C_0805_HandSoldering
- C42: renamed from C43; footprint Capacitors_SMD:C_0805 -> Capacitors_SMD:C_0805_HandSoldering
- C44: renamed from C45; footprint Capacitors_SMD:C_0805 -> Capacitors_SMD:C_0805_HandSoldering
- P1, P4, P5: footprint Pin_Headers:Pin_Header_Angled_1x02 -> Pin_Headers:Pin_Header_Straight_1x02
- P2: footprint Pin_Headers:Pin_Header_Angled_1x06 -> Pin_Headers:Pin_Header_Straight_1x06; symbol CONN_01X06 -> CONN_01X05
- R1: renamed from R99; footprint (none) -> Resistors_SMD:R_0805_HandSoldering
- R2: renamed from R98; footprint (none) -> Resistors_SMD:R_0805_HandSoldering
- U4, U5: footprint Socket_Strips:Socket_Strip_Angled_1x03 -> Pin_Headers:Pin_Header_Straight_1x03
- gave numbers to parts that had none: 1
- renumbered C23 to C22, C24 to C23, C27 to C26, C28 to C27, C37 to C36, C41 to C40, C44 to C43, C46 to C45, R12 to R10, R13 to R11, R14 to R12, R20 to R13, R21 to R14, R22 to R15, R23 to R16, R24 to R17, R25 to R19, R26 to R20, R27 to R21, R28 to R22, R29 to R23, R1 to R3, R2 to R4, R3 to R5, R4 to R6, R5 to R7, R6 to R8, R11 to R9, U11 to U10, U12 to U11, U13 to U12, U14 to U13, U15 to U14, U16 to U15, U17 to U16, U7 to U6, U8 to U7, U9 to U8, U10 to U9
Connections:
- net +3V3: now also P3.1 (P1), IC?.8 (VCC), IC?.8 (VCC); no longer P2.2 (P2)
- net +5V: now also C?.2, C?.2, U?.3 (VCC); no longer P3.1 (P1)
- net GND: now also C?.1, C?.1, IC?.4 (GND), IC?.4 (GND), P?.5 (P5), P?.5 (P5), R?.1, U?.2 (GND)
- net KILL: now also IC1.32 ((PCINT18/INT0)PD2); no longer IC1.2 ((PCINT20/XCK/T0)PD4)
- net KTIR_(1): now also IC?.2 (PB3(CLKI/ADC3/PCINT3)); no longer IC1.23 ((PCINT8/ADC0)PC0)
- net KTIR_(2): now also IC?.3 (PB4(ADC2/PCINT4)); no longer IC1.24 ((PCINT9/ADC1)PC1)
- net KTIR_(3): now also IC?.2 (PB3(CLKI/ADC3/PCINT3)); no longer IC1.25 ((PCINT10/ADC2)PC2)
- net KTIR_(4): now also IC?.3 (PB4(ADC2/PCINT4)); no longer IC1.26 ((PCINT11/ADC3)PC3)
- net MISO: now also P2.4 (P4); no longer P2.5 (P5)
- net MOSI: now also P2.3 (P3); no longer P2.4 (P4)
- net RST_328: now also P2.5 (P5); no longer P2.6 (P6)
- net SCK: now also P2.2 (P2); no longer P2.3 (P3)
- net at IC1.1 ((PCINT19/OC2B/INT1)PD3): now also U3.1 (OUT)
- new net: R?.1, U?.1 (V0)
- new net: IC?.1 (PB5(~RESET~/ADC0/PCINT5/dW)), P?.4 (P4) (x2)
- new net: IC?.6 (PB1(MISO/AIN1/OC0B/INT0/PCINT1)), P?.2 (P2) (x2)
- new net: IC?.7 (PB2(SCK/ADC1/T0/PCINT2)), P?.3 (P3) (x2)
- new net INT_KTIR1: IC1.24 ((PCINT9/ADC1)PC1), IC?.5 (PB0(MOSI/AIN0/OC0A/PCINT0)), P?.1 (P1)
- new net INT_KTIR2: IC1.25 ((PCINT10/ADC2)PC2), IC?.5 (PB0(MOSI/AIN0/OC0A/PCINT0)), P?.1 (P1)
- new net SHARP_3: IC1.23 ((PCINT8/ADC0)PC0), R?.2, R?.2
- no-connect marks 7 -> 8
Other:
- moved on the sheet: C16, C17, C18, C19, R5, R6, R7, R8, U4, U5

Commit message: 3 KTIRY
uproszczenie schematu, usunięcie 1 czujnika odległości, usunięcie 2
ATtiny13
Parts:
- removed IC? (x2): ATTINY13A-SS, SO8, symbol ATTINY13A-SS
- removed P?: PROG_A1, symbol CONN_01X05
- removed P?: PROG_A2, symbol CONN_01X05
- removed R12: 100, Resistors_SMD:R_0805_HandSoldering, symbol R
- removed R16: 10k, Resistors_SMD:R_0805_HandSoldering, symbol R
- removed U9: KTIR0711S, warsztaty:KTIR0711S, symbol KTIR0711S
- gave numbers to parts that had none: 5
- renumbered C17 to C16, C16 to C17, C18 to C19, C19 to C20, C20 to C22, C21 to C23, C22 to C24, C23 to C25, C24 to C26, C25 to C27, C26 to C28, C27 to C29, C28 to C30, C29 to C31, C30 to C32, C31 to C33, C32 to C34, C33 to C35, C34 to C36, C35 to C37, C36 to C38, C37 to C39, C38 to C40, C39 to C41, C40 to C42, C41 to C43, C42 to C44, C43 to C45, C44 to C46, C45 to C47, P4 to P6, P5 to P7, R9 to R11, R10 to R12, R11 to R13, R13 to R15, R14 to R16, R15 to R17, R17 to R19, R18 to R20, R19 to R21, R20 to R22, R21 to R23, R22 to R24, R23 to R25, R7 to R8, R8 to R9, U10 to U11, U11 to U12, U12 to U13, U13 to U14, U14 to U15, U15 to U16, U16 to U17, U5 to U4, U4 to U5, U6 to U7, U7 to U8, U8 to U9
Connections:
- net INT_KTIR1 is gone; now on net KTIR_(1): IC1.24 ((PCINT9/ADC1)PC1)
- net INT_KTIR2 is gone; now on net KTIR_(2): IC1.25 ((PCINT10/ADC2)PC2)
- net KTIR_(3): now also IC1.26 ((PCINT11/ADC3)PC3)
- no-connect marks 8 -> 7
