File: Minisumo uproszczony/Minisumo.sch (KiCad schematic (older format))
At the start: 94 parts, among them IC1 ATMEGA328P-A, P1 bateria, P2 PROGRAMATOR, P3 CONN_01X04, P6 silnik2, P7 silnik1, U1 LM1117_5V, U11 MMA7455L, U12 SFH7773, U13 74HC595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

Commit message: SCHEMAT
PCB
Connections:
- net ACC_DRDY: now also IC1.32 ((PCINT18/INT0)PD2); no longer IC1.13 ((PCINT1/OC1A)PB1)
- net ACC_INT2: now also IC1.13 ((PCINT1/OC1A)PB1); no longer IC1.32 ((PCINT18/INT0)PD2)
- net AIN_1: now also U13.5 (QF); no longer U13.4 (QE)
- net AIN_2: now also U13.4 (QE); no longer U13.5 (QF)
- net KILL: now also P3.3 (P3); no longer P3.4 (P4)
- net START: now also P3.4 (P4); no longer P3.3 (P3)
