File: Minisumo uproszczony/Minisumo.kicad_pcb (KiCad board)
At the start: 2 copper layers, 160 parts, among them IC1 ATMEGA328P-A, P1 bateria, P2 PROGRAMATOR, P3 CONN_01X04, P4 silnik2, P5 silnik1, U1 LM1117_5V, U10 KTIR0711S, U11 MMA7455L, U12 SFH7773, U13 74HC595, U14 TB6612, U15 TB6612, U16 SFH7773, U17 RGB_diode, U2 LM1117_3.3V, U3 TSOP4838, U4 SHARP_10-80, U5 SHARP_10-80, U6 LM339, U7 KTIR0711S, U8 KTIR0711S, U9 KTIR0711S, Y1 16mHz

Commit message: 3 Sharpy
dodano sharpa, dodano 2 attiny
Parts:
- removed the ? at (80.3, 90.6)
- removed the ? at (56.9, 79.6)
- removed the ? at (49.2, 75.8)
- removed the ? at (45.9, 75.9)
- removed the ? at (46.4, 70.2)
- removed the ? at (43.3, 60.5)
- removed the ? at (54.8, 45.8)
- removed the ? at (79.6, 71.9)
- removed the ? at (71.2, 53.2)
- removed the ? at (61.9, 53.0)
- removed the ? at (66.8, 66.2)
- removed the ? at (80.3, 85.8)
- removed the ? at (99.5, 53.8)
- removed the ? at (97.6, 54.1)
- removed the ? at (95.8, 54.2)
- removed the ? at (89.6, 41.0)
- removed the ? at (96.2, 25.8)
- removed the ? at (53.1, 30.9)
- removed the ? at (88.5, 64.2)
- removed the ? at (89.2, 57.7)
- removed the ? at (65.0, 72.4)
- removed the ? at (48.7, 54.1)
- removed the ? at (47.4, 50.2)
- removed the ? at (57.5, 60.6)
- removed the ? at (59.2, 72.9)
- removed the ? at (86.2, 65.9)
- removed the ? at (74.8, 61.0)
- removed the ? at (69.0, 53.5)
- removed the ? at (75.3, 59.2)
- removed the ? at (68.5, 63.7)
- removed the ? at (89.2, 50.4)
- removed the ? at (87.2, 51.7)
- removed the ? at (90.3, 64.2)
- removed the ? at (93.8, 37.1)
- removed the ? at (67.3, 58.2)
- removed the ? at (69.8, 58.2)
- removed the ? at (66.6, 55.9)
- removed the ? at (85.8, 69.2)
- removed the ? at (46.3, 61.7)
- removed the ? at (90.3, 70.0)
- removed the ? at (75.2, 74.8)
- removed the ? at (66.5, 54.1)
- removed the ? at (78.9, 65.1)
- removed the ? at (71.2, 63.0)
- removed the ? at (77.2, 49.1)
- removed the ? at (53.0, 69.2)
- removed the ? at (52.8, 73.1)
- removed the ? at (50.3, 68.8)
- removed the ? at (75.6, 70.7)
- removed the ? at (54.8, 68.7)
- removed the ? at (89.2, 48.6)
- removed the ? at (95.7, 59.1)
- removed the ? at (78.0, 42.5)
- removed the ? at (82.3, 42.6)
- removed the ? at (102.8, 36.2)
- removed the ? at (85.6, 50.8)
- removed the ? at (93.5, 66.5)
- removed C46: 100uF, Capacitors_SMD:c_elec_6.3x7.7
- removed P2: PROGRAMATOR, Pin_Headers:Pin_Header_Straight_1x05
- removed R24, R25, R27: 1k, Resistors_SMD:R_0805_HandSoldering
- removed R26, R28, R29: 220, Resistors_SMD:R_0805_HandSoldering
- removed R98, R99: 10k, Resistors_SMD:R_0805_HandSoldering
- removed U17: RGB_diode, warsztaty:RGB_C_Anode
- added ?: , Connect:PINTST, F.Cu at (58.4, 69.3)
- added ?: , Connect:PINTST, F.Cu at (78.1, 48.6)
- added ?: , Connect:PINTST, F.Cu at (76.3, 47.9)
- added ?: , Connect:PINTST, F.Cu at (74.4, 48.0)
- added ?: , Connect:PINTST, F.Cu at (96.2, 67.8)
- added ?: , Connect:PINTST, F.Cu at (84.0, 71.5)
- added ?: , Connect:PINTST, F.Cu at (89.5, 72.0)
- added ?: , Connect:PINTST, F.Cu at (93.8, 72.0)
- added ?: , Connect:PINTST, F.Cu at (78.5, 74.7)
- added ?: , Connect:PINTST, F.Cu at (81.0, 62.5)
- added ?: , Connect:PINTST, F.Cu at (73.3, 66.6)
- added ?: , Connect:PINTST, F.Cu at (77.9, 62.5)
- added ?: , Connect:PINTST, F.Cu at (49.4, 72.6)
- added ?: , Connect:PINTST, F.Cu at (52.0, 69.7)
- added ?: , Connect:PINTST, F.Cu at (56.1, 69.8)
- added ?: , Pin_Headers:Pin_Header_Straight_1x01, F.Cu at (69.0, 48.7)
- added ?: , Pin_Headers:Pin_Header_Straight_1x02, F.Cu at (43.6, 61.8)
- added ?: , Connect:PINTST, F.Cu at (79.6, 68.2)
- added ?: , Connect:PINTST, F.Cu at (89.2, 68.0)
- added ?: , Pin_Headers:Pin_Header_Straight_1x01, F.Cu at (42.9, 27.6)
- added ?: , Connect:PINTST, F.Cu at (74.0, 58.0)
- added ?: , Connect:PINTST, F.Cu at (75.8, 57.0)
- added ?: , Pin_Headers:Pin_Header_Straight_1x01, F.Cu at (83.6, 61.4)
- added ?: , Connect:PINTST, F.Cu at (49.2, 53.5)
- C1, C11, C12, C14, C15, C18, C19, C2, C20, C25, C29, C3, C30, C31, C32, C33, C34, C35, C38, C39, C4, C42, C5, C8: footprint Capacitors_SMD:C_0805 -> Capacitors_SMD:C_0805_HandSoldering
- C22: value 100nF -> 100uF; footprint Capacitors_SMD:C_0603_HandSoldering -> Capacitors_SMD:c_elec_6.3x7.7
- C23: value 100uF -> 4.7uF; footprint Capacitors_SMD:c_elec_6.3x7.7 -> Capacitors_Tantalum_SMD:TantalC_SizeA_EIA-3216_HandSoldering
- C24, C41: value 4.7uF -> 100nF; footprint Capacitors_Tantalum_SMD:TantalC_SizeA_EIA-3216_HandSoldering -> Capacitors_SMD:C_0805_HandSoldering
- C26, C43: value 100nF -> 1uF; footprint Capacitors_SMD:C_0805 -> Capacitors_Tantalum_SMD:TantalC_SizeA_EIA-3216_HandSoldering
- C27: value 1uF -> 100uF; footprint Capacitors_Tantalum_SMD:TantalC_SizeA_EIA-3216_HandSoldering -> Capacitors_SMD:c_elec_6.3x7.7
- C28, C37: value 100uF -> 100nF; footprint Capacitors_SMD:c_elec_6.3x7.7 -> Capacitors_SMD:C_0805_HandSoldering
- C36, C45: value 100nF -> 100uF; footprint Capacitors_SMD:C_0805 -> Capacitors_SMD:c_elec_6.3x7.7
- C40: value 100nF -> 4.7uF; footprint Capacitors_SMD:C_0805 -> Capacitors_Tantalum_SMD:TantalC_SizeA_EIA-3216_HandSoldering
- C44: value 1uF -> 100nF; footprint Capacitors_Tantalum_SMD:TantalC_SizeA_EIA-3216_HandSoldering -> Capacitors_SMD:C_0805_HandSoldering
- R1: value 330 -> 10K
- R10, R9: value 47K -> 100
- R13, R14: value 100 -> 10k
- R15: value 33K -> 10k
- R16: value 1K -> 10k
- R17, R18, R19: value 1K -> 1k
- R20, R22, R23: value 10k -> 220
- R21: value 10k -> 1k
- R3: value 22K -> 330
- R4: value 22K -> 10K
- R5, R6: value 6K8 -> 22K
- R7, R8: value 47K -> 6K8
- REF**: value KTIRs -> Pin_Header_Straight_2x02
- U10: value KTIR0711S -> MMA7455L; footprint warsztaty:KTIR0711S -> warsztaty:LGA_14
- U11: value MMA7455L -> SFH7773; footprint warsztaty:LGA_14 -> warsztaty:sfh7773
- U12: value SFH7773 -> 74HC595; footprint warsztaty:sfh7773 -> SMD_Packages:SO-16-N
- U13: value 74HC595 -> TB6612; footprint SMD_Packages:SO-16-N -> warsztaty:TB6612
- U15: value TB6612 -> SFH7773; footprint warsztaty:TB6612 -> warsztaty:sfh7773
- U16: value SFH7773 -> RGB_diode; footprint warsztaty:sfh7773 -> warsztaty:RGB_C_Anode
- U4, U5: footprint Socket_Strips:Socket_Strip_Straight_1x03 -> Pin_Headers:Pin_Header_Straight_1x03
- U6: value LM339 -> KTIR0711S; footprint warsztaty:SO14 -> warsztaty:KTIR0711S
- moved R22 163.7 mm to (64.4, 70.7)
- moved R23 156.8 mm to (64.5, 68.6)
- moved U10 139.0 mm to (84.8, 47.5)
- moved U16 121.3 mm to (44.2, 96.3), turned to 90 degrees
- moved R15 120.0 mm to (207.9, 67.1), turned to 0 degrees
- moved R19 108.6 mm to (197.1, 92.6)
- moved R16 108.0 mm to (213.0, 60.8), turned to 0 degrees
- moved R9 107.2 mm to (197.1, 80.0), turned to 0 degrees
- moved R10 105.8 mm to (190.0, 86.3), turned to 0 degrees
- moved R20 105.7 mm to (64.4, 72.8)
- moved C27 103.8 mm to (45.2, 87.9), turned to 90 degrees
- moved U15 101.0 mm to (153.3, 64.3), turned to 0 degrees
- moved U6 96.3 mm to (194.2, 61.4)
- moved C40 95.7 mm to (154.6, 94.7), turned to 0 degrees
- moved C25 90.7 mm to (210.6, 54.5)
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Connections:
- C2 pad 1: VCC -> +5V
- C22 pad 1: /POROWNANIE -> +5V
- C23 pad 1: +5V -> +3V3
- C24 pad 1: +3V3 -> GND
- C24 pad 2: GND -> +3V3
- C25 pad 1: GND -> +3V3
- C25 pad 2: +3V3 -> GND
- C27 pad 1: +3V3 -> +5V
- C28 pad 1: +5V -> GND
- C28 pad 2: GND -> +5V
- C34 pad 2: +5V -> VCC
- C36 pad 1: GND -> VCC
- C36 pad 2: VCC -> GND
- C37 pad 1: VCC -> GND
- C37 pad 2: GND -> VCC
- C40 pad 1: GND -> +3V3
- C40 pad 2: VCC -> GND
- C41 pad 1: +3V3 -> GND
- C41 pad 2: GND -> +3V3
- C42 pad 1: GND -> +3V3
- C42 pad 2: +3V3 -> GND
- C44 pad 1: +3V3 -> GND
- C44 pad 2: GND -> VCC
- C45 pad 1: GND -> VCC
- C45 pad 2: VCC -> GND
- C7 pad 1: VCC -> +5V
- IC1 pad 1: /KTIR_PWM -> Net-(IC1-Pad1)
- IC1 pad 2: /KILL -> Net-(IC1-Pad2)
- IC1 pad 23: /INT_KTIR_2 -> /KTIR_(1)
- IC1 pad 24: /INT_KTIR_1 -> /KTIR_(2)
- IC1 pad 25: /INT_KTIR_3 -> /KTIR_(3)
- IC1 pad 26: /INT_KTIR_4 -> /KTIR_(4)
- IC1 pad 32: Net-(IC1-Pad32) -> /KILL
- R1 pad 1: Net-(C13-Pad1) -> +3V3
- R1 pad 2: +3V3 -> /SDA
- R10 pad 2: /INT_KTIR_4 -> +3V3
- R13 pad 1: Net-(R13-Pad1) -> +3V3
- R13 pad 2: +3V3 -> /KTIR_(1)
- R14 pad 1: Net-(R14-Pad1) -> +3V3
- R14 pad 2: +3V3 -> /KTIR_(2)
- R15 pad 1: /POROWNANIE -> +3V3
- R15 pad 2: /KTIR_PWM -> /KTIR_(3)
- R16 pad 1: /POROWNANIE -> +3V3
- R16 pad 2: Net-(R16-Pad2) -> /KTIR_(4)
- R17 pad 1: /POROWNANIE -> /ACC_INT2
- R18 pad 1: /POROWNANIE -> /ACC_DRDY
- R19 pad 1: /POROWNANIE -> Net-(R19-Pad1)
- R19 pad 2: Net-(R10-Pad1) -> /INT_10_2
- R2 pad 2: /RST_328 -> /SCL
- R20 pad 1: +3V3 -> Net-(R20-Pad1)
- R20 pad 2: /KTIR_(1) -> Net-(R20-Pad2)
- R21 pad 1: +3V3 -> Net-(R21-Pad1)
- R21 pad 2: /KTIR_(2) -> /INT_10_1
- R22 pad 1: +3V3 -> Net-(R22-Pad1)
- R22 pad 2: /KTIR_(3) -> Net-(R22-Pad2)
- R23 pad 1: +3V3 -> Net-(R23-Pad1)
- R23 pad 2: /KTIR_(4) -> Net-(R23-Pad2)
- R3 pad 1: GND -> Net-(C13-Pad1)
- R3 pad 2: /SHARP_1 -> +3V3
- R4 pad 1: GND -> +3V3
- R4 pad 2: /SHARP_2 -> /RST_328
- R5 pad 1: Net-(R5-Pad1) -> GND
- R6 pad 1: Net-(R6-Pad1) -> GND
- R7 pad 1: Net-(R16-Pad2) -> Net-(R7-Pad1)
- R7 pad 2: /INT_KTIR_1 -> /SHARP_1
- R8 pad 1: Net-(R17-Pad2) -> Net-(R8-Pad1)
- R8 pad 2: /INT_KTIR_2 -> /SHARP_2
- R9 pad 1: Net-(R18-Pad2) -> Net-(R9-Pad1)
- R9 pad 2: /INT_KTIR_3 -> +3V3
- U1 pad 4: GND -> (no net)
- U10 pad 1: Net-(R14-Pad1) -> +3V3
- U10 pad 4: /KTIR_(4) -> +3V3
- U11 pad 3: GND -> +3V3
- U11 pad 4: +3V3 -> GND
- U11 pad 5: GND -> Net-(R19-Pad1)
- U11 pad 6: +3V3 -> /SCL
- U11 pad 7: +3V3 -> /SDA
- U11 pad 8: /ACC_DRDY -> Net-(U11-Pad8)
- U12 pad 1: +3V3 -> Net-(R23-Pad2)
- U12 pad 2: GND -> Net-(R22-Pad2)
- U12 pad 3: +3V3 -> Net-(R20-Pad2)
- U12 pad 4: GND -> /AIN_1
- U12 pad 5: Net-(R25-Pad1) -> /AIN_2
- U12 pad 6: /SCL -> /BIN_1
- U12 pad 7: /SDA -> /BIN_2
- U12 pad 8: Net-(U12-Pad8) -> GND
- U13 pad 1: Net-(R26-Pad2) -> /S_B_1
- U13 pad 10: +3V3 -> GND
- U13 pad 11: /SCK -> /S_B_1
- U13 pad 12: /SS -> /S_B_1
- U13 pad 13: GND -> VCC
- U13 pad 14: /MOSI -> VCC
- U13 pad 15: Net-(U13-Pad15) -> /PWM_B
- U13 pad 16: +3V3 -> /BIN_2
- U13 pad 2: Net-(R28-Pad2) -> /S_B_1
- U13 pad 3: Net-(R29-Pad2) -> GND
- U13 pad 4: /AIN_1 -> GND
- U13 pad 5: /AIN_2 -> /S_B_2
- U13 pad 6: /BIN_1 -> /S_B_2
- U13 pad 7: /BIN_2 -> /S_B_2
- U13 pad 8: GND -> /S_B_2
- U13 pad 9: Net-(U13-Pad9) -> GND
- U14 pad 1: /S_B_1 -> /S_A_1
- U14 pad 11: /S_B_1 -> /S_A_1
- U14 pad 12: /S_B_1 -> /S_A_1
- U14 pad 15: /PWM_B -> /PWM_A
- U14 pad 16: /BIN_2 -> /AIN_2
- U14 pad 17: /BIN_1 -> /AIN_1
- U14 pad 2: /S_B_1 -> /S_A_1
- U14 pad 21: /BIN_2 -> /AIN_2
- U14 pad 22: /BIN_1 -> /AIN_1
- U14 pad 23: /PWM_B -> /PWM_A
- U14 pad 5: /S_B_2 -> /S_A_2
- U14 pad 6: /S_B_2 -> /S_A_2
- U14 pad 7: /S_B_2 -> /S_A_2
- U14 pad 8: /S_B_2 -> /S_A_2
- U15 pad 1: /S_A_1 -> +3V3
- U15 pad 2: /S_A_1 -> GND
- U15 pad 3: GND -> +3V3
- U15 pad 5: /S_A_2 -> Net-(R21-Pad1)
- U15 pad 6: /S_A_2 -> /SCL
- U15 pad 7: /S_A_2 -> /SDA
- U15 pad 8: /S_A_2 -> Net-(U15-Pad8)
- U16 pad 1: +3V3 -> Net-(R20-Pad1)
- U16 pad 2: GND -> +5V
- U16 pad 3: +3V3 -> Net-(R22-Pad1)
- U16 pad 4: GND -> Net-(R23-Pad1)
- U2 pad 1: VCC -> +5V
- U3 pad 1: Net-(IC1-Pad32) -> Net-(IC1-Pad1)
- U4 pad 1: Net-(R6-Pad1) -> Net-(R8-Pad1)
- U5 pad 1: Net-(R5-Pad1) -> Net-(R7-Pad1)
- U6 pad 1: /INT_KTIR_1 -> Net-(R9-Pad1)
- U6 pad 2: /INT_KTIR_2 -> GND
- U6 pad 3: +3V3 -> GND
- U6 pad 4: Net-(R16-Pad2) -> /KTIR_(1)
- U7 pad 1: Net-(R11-Pad1) -> Net-(R10-Pad1)
- U7 pad 4: /KTIR_(1) -> /KTIR_(2)
- U8 pad 1: Net-(R12-Pad1) -> Net-(R11-Pad1)
- U8 pad 4: /KTIR_(2) -> /KTIR_(3)
- U9 pad 1: Net-(R13-Pad1) -> Net-(R12-Pad1)
- U9 pad 4: /KTIR_(3) -> /KTIR_(4)
- Y1 pad 1: /XTAL2 -> /XTAL1
- Y1 pad 2: /XTAL1 -> /XTAL2
Routing:
- net VCC: track 359.9 -> 142.8 mm
- net +5V: track 386.8 -> 201.4 mm
- net GND: track 223.4 -> 80.0 mm
- net +3V3: track 247.4 -> 108.1 mm
- net /RST_328: track 92.9 -> 33.8 mm
- net Net-(R20-Pad1): track 0.00 -> 46.4 mm
- net /SCK: track 58.5 -> 12.8 mm
- net /MOSI: track 86.2 -> 41.0 mm
- net Net-(R29-Pad1): track 38.3 -> 0.00 mm
- net /ACC_DRDY: track 38.1 -> 0.00 mm
- net Net-(R22-Pad1): track 0.00 -> 35.9 mm
- net /INT_KTIR_4: track 35.3 -> 0.00 mm
- net Net-(R23-Pad1): track 0.00 -> 34.5 mm
- net Net-(R5-Pad1): track 34.0 -> 0.00 mm
- net Net-(R26-Pad1): track 33.1 -> 0.00 mm
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
Commit message: SCHEMAT
PCB
Parts:
- removed the ? at (58.4, 69.3)
- removed the ? at (78.1, 48.6)
- removed the ? at (76.3, 47.9)
- removed the ? at (74.4, 48.0)
- removed the ? at (96.2, 67.8)
- removed the ? at (84.0, 71.5)
- removed the ? at (89.5, 72.0)
- removed the ? at (93.8, 72.0)
- removed the ? at (78.5, 74.7)
- removed the ? at (81.0, 62.5)
- removed the ? at (73.3, 66.6)
- removed the ? at (77.9, 62.5)
- removed the ? at (49.4, 72.6)
- removed the ? at (52.0, 69.7)
- removed the ? at (56.1, 69.8)
- removed the ? at (69.0, 48.7)
- removed the ? at (43.6, 61.8)
- removed the ? at (79.6, 68.2)
- removed the ? at (89.2, 68.0)
- removed the ? at (42.9, 27.6)
- removed the ? at (74.0, 58.0)
- removed the ? at (75.8, 57.0)
- removed the ? at (83.6, 61.4)
- removed the ? at (49.2, 53.5)
- removed P4: silnik2, Pin_Headers:Pin_Header_Straight_1x02
- removed P5: silnik1, Pin_Headers:Pin_Header_Straight_1x02
- removed R14: 10k, Resistors_SMD:R_0805_HandSoldering
- removed R18: 1k, Resistors_SMD:R_0805_HandSoldering
- removed U10: MMA7455L, warsztaty:LGA_14
- added ?: , Connect:PINTST, F.Cu at (75.7, 146.8)
- added ?: , Pin_Headers:Pin_Header_Straight_1x02, F.Cu at (126.5, 96.0)
- added ?: , Connect:PINTST, F.Cu at (92.8, 149.0)
- added ?: , Connect:PINTST, F.Cu at (109.2, 129.0)
- added ?: , Connect:PINTST, F.Cu at (95.8, 139.6)
- added ?: , Connect:PINTST, F.Cu at (97.1, 143.1)
- added ?: , Connect:PINTST, F.Cu at (94.8, 144.5)
- added ?: , Connect:PINTST, F.Cu at (95.5, 148.9)
- added ?: , Connect:PINTST, F.Cu at (102.0, 158.3)
- added ?: , Connect:PINTST, F.Cu at (80.3, 146.8)
- added ?: , Connect:PINTST, F.Cu at (100.8, 135.1)
- added ?: , Pin_Headers:Pin_Header_Straight_1x03, F.Cu at (105.0, 61.5)
- added ?: , Connect:PINTST, F.Cu at (124.8, 172.4)
- added ?: , Connect:PINTST, F.Cu at (122.9, 168.3)
- added ?: , Connect:PINTST, F.Cu at (106.9, 151.7)
- added ?: , Connect:PINTST, F.Cu at (81.9, 142.7)
- added ?: , Connect:PINTST, F.Cu at (83.2, 157.0)
- added ?: , Connect:PINTST, F.Cu at (99.6, 127.6)
- added ?: , Connect:PINTST, F.Cu at (73.1, 139.2)
- added ?: , Connect:PINTST, F.Cu at (66.0, 164.4)
- added ?: , Connect:PINTST, F.Cu at (100.1, 147.1)
- added ?: , Connect:PINTST, F.Cu at (94.4, 133.6)
- added ?: , Pin_Headers:Pin_Header_Straight_1x02, F.Cu at (75.0, 63.0)
- added ?: , Connect:PINTST, F.Cu at (77.8, 168.9)
- added ?: , Connect:PINTST, F.Cu at (75.7, 168.9)
- added ?: , Connect:PINTST, F.Cu at (72.8, 164.7)
- added ?: , Connect:PINTST, F.Cu at (70.3, 164.6)
- added ?: , Connect:PINTST, F.Cu at (72.5, 155.5)
- added ?: , Connect:PINTST, F.Cu at (114.8, 155.8)
- added ?: , Connect:PINTST, F.Cu at (113.1, 152.4)
- added ?: , Connect:PINTST, F.Cu at (115.0, 152.9)
- added ?: , Connect:PINTST, F.Cu at (93.1, 144.4)
- added ?: , Connect:PINTST, F.Cu at (97.9, 148.4)
- added ?: , Pin_Headers:Pin_Header_Straight_1x02, F.Cu at (75.0, 75.0)
- added ?: , Connect:PINTST, F.Cu at (94.2, 152.7)
- added ?: , Connect:PINTST, F.Cu at (82.0, 151.7)
- added ?: , Connect:PINTST, F.Cu at (80.2, 151.7)
- added ?: , Pin_Headers:Pin_Header_Straight_2x05, F.Cu at (68.2, 180.1)
- added ?: , Pin_Headers:Pin_Header_Straight_1x02, F.Cu at (68.5, 96.0)
- added ?: , Pin_Headers:Pin_Header_Straight_1x03, F.Cu at (105.0, 73.5)
- added ?: , Connect:PINTST, F.Cu at (99.0, 135.7)
- added ?: , Connect:PINTST, F.Cu at (97.9, 134.1)
- added ?: , Pin_Headers:Pin_Header_Straight_1x02, F.Cu at (126.5, 86.0)
- added ?: , Pin_Headers:Pin_Header_Straight_1x02, F.Cu at (68.5, 86.0)
- added ?: , Connect:PINTST, F.Cu at (94.2, 168.7)
- added C46: 100nF, Capacitors_SMD:C_0805_HandSoldering, F.Cu at (113.4, 147.6)
- added C47: 100uF, Capacitors_SMD:c_elec_6.3x7.7, F.Cu at (85.4, 164.8)
- added P2: PROGRAMATOR, Pin_Headers:Pin_Header_Straight_1x05, F.Cu at (71.9, 180.1)
- added P6: silnik2, Pin_Headers:Pin_Header_Straight_1x02, F.Cu at (128.3, 152.2)
- added P7: silnik1, Pin_Headers:Pin_Header_Straight_1x02, F.Cu at (66.6, 149.7)
- added R24: 220, Resistors_SMD:R_0805_HandSoldering, F.Cu at (94.0, 163.0)
- added R25: 220, Resistors_SMD:R_0805_HandSoldering, F.Cu at (96.3, 163.0)
- added REF**: Pin_Header_Straight_1x03, Pin_Headers:Pin_Header_Straight_1x03, F.Cu at (91.9, 121.9)
- added U17: RGB_diode, warsztaty:RGB_C_Anode, F.Cu at (101.1, 164.8)
- C18: value 100nF -> 1uF; footprint Capacitors_SMD:C_0805_HandSoldering -> Capacitors_Elko_ThroughHole:Elko_vert_11x5mm_RM2
- C21: value 22uF -> 100nF; footprint Capacitors_SMD:c_elec_4x4.5 -> Capacitors_SMD:C_0805_HandSoldering
- C22, C27, C36: value 100uF -> 100nF; footprint Capacitors_SMD:c_elec_6.3x7.7 -> Capacitors_SMD:C_0805_HandSoldering
- C23: value 4.7uF -> 22uF; footprint Capacitors_Tantalum_SMD:TantalC_SizeA_EIA-3216_HandSoldering -> Capacitors_SMD:c_elec_4x4.5
- C24, C29, C38: value 100nF -> 100uF; footprint Capacitors_SMD:C_0805_HandSoldering -> Capacitors_SMD:c_elec_6.3x7.7
- C25, C42: value 100nF -> 4.7uF; footprint Capacitors_SMD:C_0805_HandSoldering -> Capacitors_Tantalum_SMD:TantalC_SizeA_EIA-3216_HandSoldering
- C26, C43: value 1uF -> 100nF; footprint Capacitors_Tantalum_SMD:TantalC_SizeA_EIA-3216_HandSoldering -> Capacitors_SMD:C_0805_HandSoldering
- C28: value 100nF -> 1uF; footprint Capacitors_SMD:C_0805_HandSoldering -> Capacitors_Tantalum_SMD:TantalC_SizeA_EIA-3216_HandSoldering
- C40: value 4.7uF -> 100nF; footprint Capacitors_Tantalum_SMD:TantalC_SizeA_EIA-3216_HandSoldering -> Capacitors_SMD:C_0805_HandSoldering
- C45: value 100uF -> 1uF; footprint Capacitors_SMD:c_elec_6.3x7.7 -> Capacitors_Tantalum_SMD:TantalC_SizeA_EIA-3216_HandSoldering
- R10, R9: value 100 -> 6K8
- R13: value 10k -> 100
- R17: value 1k -> 10k
- R20, R23: value 220 -> 1k
- R7: value 6K8 -> 22K
- REF**: value Pin_Header_Straight_2x02 -> Pin_Header_Straight_1x02
- U11: value SFH7773 -> MMA7455L; footprint warsztaty:sfh7773 -> warsztaty:LGA_14
- U12: value 74HC595 -> SFH7773; footprint SMD_Packages:SO-16-N -> warsztaty:sfh7773
- U13: value TB6612 -> 74HC595; footprint warsztaty:TB6612 -> SMD_Packages:SO-16-N
- U15: value SFH7773 -> TB6612; footprint warsztaty:sfh7773 -> warsztaty:TB6612
- U16: value RGB_diode -> SFH7773; footprint warsztaty:RGB_C_Anode -> warsztaty:sfh7773
- U6: value KTIR0711S -> SHARP_10-80; footprint warsztaty:KTIR0711S -> Pin_Headers:Pin_Header_Straight_1x03
- moved C9 151.9 mm to (127.2, 181.4), turned to 90 degrees
- moved C1 146.5 mm to (117.2, 168.3), turned to 0 degrees
- moved R11 143.2 mm to (84.0, 99.0)
- moved U1 140.3 mm to (110.0, 165.3), turned to 90 degrees
- moved C11 137.8 mm to (115.8, 162.5), turned to 90 degrees
- moved C6 133.8 mm to (127.2, 171.4)
- moved C25 127.1 mm to (85.5, 76.3), turned to 90 degrees
- moved R15 127.0 mm to (84.0, 95.0), turned to 180 degrees
- moved C43 122.4 mm to (82.8, 64.2), turned to 270 degrees
- moved R12 122.3 mm to (112.3, 95.7), turned to 180 degrees
- moved C42 118.9 mm to (97.5, 64.8), turned to 270 degrees
- moved U15 118.7 mm to (74.0, 152.6)
- moved C24 118.2 mm to (126.2, 160.4), turned to 180 degrees
- moved R21 118.2 mm to (93.2, 73.4)
- moved R1 116.9 mm to (95.9, 131.4)
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Connections:
- C20 pad 2: +3V3 -> +5V
- C21 pad 1: +3V3 -> GND
- C21 pad 2: GND -> +5V
- C22 pad 1: +5V -> GND
- C22 pad 2: GND -> +3V3
- C24 pad 1: GND -> +5V
- C24 pad 2: +3V3 -> GND
- C26 pad 1: +3V3 -> GND
- C26 pad 2: GND -> +3V3
- C27 pad 1: +5V -> +3V3
- C28 pad 1: GND -> +3V3
- C28 pad 2: +5V -> GND
- C29 pad 1: GND -> +5V
- C29 pad 2: +5V -> GND
- C34 pad 2: VCC -> +5V
- C35 pad 2: VCC -> +5V
- C36 pad 1: VCC -> GND
- C36 pad 2: GND -> VCC
- C38 pad 1: GND -> VCC
- C38 pad 2: VCC -> GND
- C40 pad 1: +3V3 -> GND
- C40 pad 2: GND -> VCC
- C41 pad 2: +3V3 -> VCC
- C43 pad 1: +3V3 -> GND
- C43 pad 2: GND -> +3V3
- C44 pad 1: GND -> +3V3
- C44 pad 2: VCC -> GND
- C45 pad 1: VCC -> +3V3
- IC1 pad 13: /ACC_DRDY -> /ACC_INT2
- IC1 pad 23: /KTIR_(1) -> /SHARP_3
- IC1 pad 24: /KTIR_(2) -> /KTIR_(1)
- IC1 pad 25: /KTIR_(3) -> /KTIR_(2)
- IC1 pad 26: /KTIR_(4) -> /KTIR_(3)
- IC1 pad 30: /ACC_INT2 -> /KILL
- IC1 pad 32: /KILL -> /ACC_DRDY
- P3 pad 1: +5V -> +3V3
- P3 pad 3: /START -> /KILL
- P3 pad 4: /KILL -> /START
- R10 pad 2: +3V3 -> /SHARP_3
- R13 pad 1: +3V3 -> Net-(R13-Pad1)
- R13 pad 2: /KTIR_(1) -> +3V3
- R15 pad 2: /KTIR_(3) -> /KTIR_(1)
- R16 pad 2: /KTIR_(4) -> /KTIR_(2)
- R17 pad 1: /ACC_INT2 -> +3V3
- R17 pad 2: Net-(R17-Pad2) -> /KTIR_(3)
- R19 pad 1: Net-(R19-Pad1) -> /ACC_INT2
- R19 pad 2: /INT_10_2 -> Net-(R19-Pad2)
- R20 pad 1: Net-(R20-Pad1) -> /ACC_DRDY
- R21 pad 2: /INT_10_1 -> /INT_10_2
- R23 pad 2: Net-(R23-Pad2) -> /INT_10_1
- R7 pad 1: Net-(R7-Pad1) -> GND
- R7 pad 2: /SHARP_1 -> /SHARP_3
- R8 pad 2: /SHARP_2 -> /SHARP_1
- R9 pad 2: +3V3 -> /SHARP_2
- REF** pad 1: /KTIR_(3) -> /SCL
- REF** pad 2: /KTIR_(4) -> /SCL
- REF** pad 3: /KTIR_(2) -> /SDA
- REF** pad 4: /KTIR_(1) -> /SDA
- U11 pad 3: +3V3 -> GND
- U11 pad 4: GND -> +3V3
- U11 pad 5: Net-(R19-Pad1) -> GND
- U11 pad 6: /SCL -> +3V3
- U11 pad 7: /SDA -> +3V3
- U11 pad 8: Net-(U11-Pad8) -> Net-(R20-Pad2)
- U12 pad 1: Net-(R23-Pad2) -> +3V3
- U12 pad 2: Net-(R22-Pad2) -> GND
- U12 pad 3: Net-(R20-Pad2) -> +3V3
- U12 pad 4: /AIN_1 -> GND
- U12 pad 5: /AIN_2 -> Net-(R21-Pad1)
- U12 pad 6: /BIN_1 -> /SCL
- U12 pad 7: /BIN_2 -> /SDA
- U12 pad 8: GND -> Net-(U12-Pad8)
- U13 pad 1: /S_B_1 -> Net-(R22-Pad2)
- U13 pad 10: GND -> +3V3
- U13 pad 11: /S_B_1 -> /SCK
- U13 pad 12: /S_B_1 -> /SS
- U13 pad 13: VCC -> GND
- U13 pad 14: VCC -> /MOSI
- U13 pad 15: /PWM_B -> Net-(U13-Pad15)
- U13 pad 16: /BIN_2 -> +3V3
- U13 pad 2: /S_B_1 -> Net-(R24-Pad2)
- U13 pad 3: GND -> Net-(R25-Pad2)
- U13 pad 4: GND -> /AIN_2
- U13 pad 5: /S_B_2 -> /AIN_1
- U13 pad 6: /S_B_2 -> /BIN_1
- U13 pad 7: /S_B_2 -> /BIN_2
- U13 pad 8: /S_B_2 -> GND
- U13 pad 9: GND -> Net-(U13-Pad9)
- U14 pad 1: /S_A_1 -> /S_B_1
- U14 pad 11: /S_A_1 -> /S_B_1
- U14 pad 12: /S_A_1 -> /S_B_1
- U14 pad 15: /PWM_A -> /PWM_B
- U14 pad 16: /AIN_2 -> /BIN_2
- U14 pad 17: /AIN_1 -> /BIN_1
- U14 pad 2: /S_A_1 -> /S_B_1
- U14 pad 21: /AIN_2 -> /BIN_2
- U14 pad 22: /AIN_1 -> /BIN_1
- U14 pad 23: /PWM_A -> /PWM_B
- U14 pad 5: /S_A_2 -> /S_B_2
- U14 pad 6: /S_A_2 -> /S_B_2
- U14 pad 7: /S_A_2 -> /S_B_2
- U14 pad 8: /S_A_2 -> /S_B_2
- U15 pad 1: +3V3 -> /S_A_1
- U15 pad 2: GND -> /S_A_1
- U15 pad 3: +3V3 -> GND
- U15 pad 5: Net-(R21-Pad1) -> /S_A_2
- U15 pad 6: /SCL -> /S_A_2
- U15 pad 7: /SDA -> /S_A_2
- U15 pad 8: Net-(U15-Pad8) -> /S_A_2
- U16 pad 1: Net-(R20-Pad1) -> +3V3
- U16 pad 2: +5V -> GND
- U16 pad 3: Net-(R22-Pad1) -> +3V3
- U16 pad 4: Net-(R23-Pad1) -> GND
- U5 pad 1: Net-(R7-Pad1) -> Net-(R9-Pad1)
- U6 pad 1: Net-(R9-Pad1) -> Net-(R10-Pad1)
- U6 pad 3: GND -> +5V
- U7 pad 1: Net-(R10-Pad1) -> Net-(R11-Pad1)
- U7 pad 4: /KTIR_(2) -> /KTIR_(1)
- U8 pad 1: Net-(R11-Pad1) -> Net-(R12-Pad1)
- U8 pad 4: /KTIR_(3) -> /KTIR_(2)
- U9 pad 1: Net-(R12-Pad1) -> Net-(R13-Pad1)
- U9 pad 4: /KTIR_(4) -> /KTIR_(3)
Routing:
- net +3V3: track 108.1 -> 476.4 mm
- net GND: track 80.0 -> 339.7 mm
- net +5V: track 201.4 -> 304.5 mm
- net /SCL: track 11.2 -> 78.6 mm
- net /SCK: track 12.8 -> 74.2 mm
- net /INT_10_1: track 0.00 -> 61.0 mm
- net /INT_10_2: track 0.00 -> 60.1 mm
- net /SDA: track 9.86 -> 65.9 mm
- net Net-(R20-Pad1): track 46.4 -> 0.00 mm
- net /KTIR_(3): track 5.33 -> 49.9 mm
- net /KTIR_(1): track 8.46 -> 50.9 mm
- net VCC: track 142.8 -> 184.1 mm
- net /KTIR_(2): track 4.07 -> 41.8 mm
- net Net-(R9-Pad1): track 0.00 -> 33.2 mm
- net Net-(R23-Pad1): track 34.5 -> 2.20 mm
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
Commit message: poprawione PCB
PCB v2
Parts:
- removed the ? at (75.7, 146.8)
- removed the ? at (92.8, 149.0)
- removed the ? at (109.2, 129.0)
- removed the ? at (95.8, 139.6)
- removed the ? at (97.1, 143.1)
- removed the ? at (94.8, 144.5)
- removed the ? at (95.5, 148.9)
- removed the ? at (102.0, 158.3)
- removed the ? at (80.3, 146.8)
- removed the ? at (100.8, 135.1)
- removed the ? at (124.8, 172.4)
- removed the ? at (122.9, 168.3)
- removed the ? at (106.9, 151.7)
- removed the ? at (81.9, 142.7)
- removed the ? at (83.2, 157.0)
- removed the ? at (99.6, 127.6)
- removed the ? at (73.1, 139.2)
- removed the ? at (66.0, 164.4)
- removed the ? at (100.1, 147.1)
- removed the ? at (94.4, 133.6)
- removed the ? at (77.8, 168.9)
- removed the ? at (75.7, 168.9)
- removed the ? at (72.8, 164.7)
- removed the ? at (70.3, 164.6)
- removed the ? at (72.5, 155.5)
- removed the ? at (114.8, 155.8)
- removed the ? at (113.1, 152.4)
- removed the ? at (115.0, 152.9)
- removed the ? at (93.1, 144.4)
- removed the ? at (97.9, 148.4)
- removed the ? at (94.2, 152.7)
- removed the ? at (82.0, 151.7)
- removed the ? at (80.2, 151.7)
- removed the ? at (99.0, 135.7)
- removed the ? at (97.9, 134.1)
- removed the ? at (94.2, 168.7)
- added ?: , Connect:PINTST, F.Cu at (115.0, 178.0)
- added ?: , Connect:PINTST, F.Cu at (74.8, 169.9)
- added ?: , Connect:PINTST, F.Cu at (111.5, 184.0)
- added ?: , Connect:PINTST, F.Cu at (85.5, 171.7)
- added ?: , Connect:PINTST, F.Cu at (111.7, 178.8)
- added ?: , Connect:PINTST, F.Cu at (109.5, 171.4)
- added ?: , Connect:PINTST, F.Cu at (87.3, 166.2)
- added ?: , Connect:PINTST, F.Cu at (122.8, 186.4)
- added ?: , Connect:PINTST, F.Cu at (124.2, 184.3)
- added ?: , Connect:PINTST, F.Cu at (113.2, 176.5)
- added ?: , Connect:PINTST, F.Cu at (108.7, 143.3)
- added ?: , Connect:PINTST, F.Cu at (81.2, 163.8)
- added ?: , Connect:PINTST, F.Cu at (104.2, 144.2)
- added ?: , Connect:PINTST, F.Cu at (105.1, 142.6)
- added ?: , Connect:PINTST, F.Cu at (106.1, 144.2)
- added ?: , Connect:PINTST, F.Cu at (97.2, 145.9)
- added ?: , Connect:PINTST, F.Cu at (75.8, 125.8)
- added ?: , Connect:PINTST, F.Cu at (108.2, 150.8)
- added ?: , Connect:PINTST, F.Cu at (115.2, 128.9)
- added ?: , Connect:PINTST, F.Cu at (114.8, 134.1)
- added ?: , Connect:PINTST, F.Cu at (84.0, 126.5)
- added ?: , Connect:PINTST, F.Cu at (93.3, 141.3)
- added ?: , Connect:PINTST, F.Cu at (81.9, 154.1)
- added ?: , Connect:PINTST, F.Cu at (109.7, 152.3)
- added ?: , Connect:PINTST, F.Cu at (94.2, 146.3)
- added ?: , Connect:PINTST, F.Cu at (106.7, 152.4)
- added ?: , Connect:PINTST, F.Cu at (94.3, 148.4)
- added ?: , Connect:PINTST, F.Cu at (93.8, 150.3)
- added ?: , Connect:PINTST, F.Cu at (74.9, 165.8)
- added ?: , Connect:PINTST, F.Cu at (75.7, 157.4)
- added ?: , Connect:PINTST, F.Cu at (75.6, 152.3)
- added ?: , Connect:PINTST, F.Cu at (76.7, 170.4)
- added ?: , Connect:PINTST, F.Cu at (72.5, 186.2)
- added ?: , Connect:PINTST, F.Cu at (83.2, 156.0)
- added ?: , Connect:PINTST, F.Cu at (83.4, 143.7)
- added ?: , Connect:PINTST, F.Cu at (81.8, 142.8)
- added ?: , Connect:PINTST, F.Cu at (79.0, 144.6)
- added ?: , Connect:PINTST, F.Cu at (88.0, 151.4)
- added ?: , Connect:PINTST, F.Cu at (119.3, 126.2)
- added ?: , Connect:PINTST, F.Cu at (120.7, 133.7)
- added ?: , Connect:PINTST, F.Cu at (114.8, 132.2)
- added ?: , Connect:PINTST, F.Cu at (88.8, 146.2)
- added ?: , Connect:PINTST, F.Cu at (78.3, 126.2)
- added ?: , Connect:PINTST, F.Cu at (78.6, 131.2)
- added ?: , Connect:PINTST, F.Cu at (121.0, 155.8)
- added ?: , Connect:PINTST, F.Cu at (87.9, 144.4)
- added ?: , Connect:PINTST, F.Cu at (80.4, 131.8)
- added ?: , Connect:PINTST, F.Cu at (117.9, 149.6)
- added ?: , Connect:PINTST, F.Cu at (87.2, 142.7)
- added ?: , Pin_Headers:Pin_Header_Straight_1x01, F.Cu at (88.1, 130.6)
- added ?: , Connect:PINTST, F.Cu at (124.9, 152.8)
- added ?: , Connect:PINTST, F.Cu at (97.9, 153.6)
- added ?: , Connect:PINTST, F.Cu at (102.3, 170.9)
- added P3: CONN_01X04, Pin_Headers:Pin_Header_Straight_1x02, F.Cu at (88.5, 163.3)
- ?: footprint Pin_Headers:Pin_Header_Straight_2x05 -> Pin_Headers:Pin_Header_Straight_2x04
- moved U5 76.1 mm to (66.9, 166.5), turned to 180 degrees
- moved U6 75.4 mm to (66.9, 175.3)
- moved C18 67.4 mm to (71.3, 173.8), turned to 270 degrees
- moved C21 67.3 mm to (71.2, 171.1), turned to 0 degrees
- moved R20 66.9 mm to (127.7, 184.2)
- moved U4 63.9 mm to (67.0, 152.7), turned to 0 degrees
- moved C20 61.6 mm to (71.3, 162.3), turned to 0 degrees
- moved C9 61.4 mm to (93.7, 129.9)
- moved ? 59.9 mm to (127.3, 171.2)
- moved R19 59.8 mm to (126.3, 186.6), turned to 0 degrees
- moved R1 58.8 mm to (119.2, 185.4)
- moved R2 58.6 mm to (119.2, 183.1)
- moved C17 57.5 mm to (71.3, 165.0), turned to 270 degrees
- moved C22 57.1 mm to (122.2, 180.1), turned to 270 degrees
- moved U11 56.1 mm to (127.0, 180.6), turned to 0 degrees
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Connections:
- ? pad 7: /INT_10_2 -> +3V3
- P2 pad 1: GND -> /RST_328
- P2 pad 3: /MOSI -> /MISO
- P2 pad 4: /MISO -> /MOSI
- P2 pad 5: /RST_328 -> GND
- P3 pad 1: +3V3 -> GND
- P3 pad 2: GND -> +3V3
- REF** pad 1: /KTIR_(1) -> /KTIR_(3)
- REF** pad 3: /KTIR_(3) -> /KTIR_(1)
Routing:
- net GND: track 339.7 -> 569.3 mm
- net /SHARP_2: track 9.40 -> 84.7 mm
- net /SHARP_3: track 16.8 -> 89.5 mm
- net /SHARP_1: track 19.3 -> 89.9 mm
- net +3V3: track 476.4 -> 413.4 mm
- net /SDA: track 65.9 -> 128.8 mm
- net Net-(R25-Pad2): track 5.44 -> 65.9 mm
- net +5V: track 304.5 -> 246.3 mm
- net /ACC_INT2: track 33.4 -> 90.6 mm
- net /SCL: track 78.6 -> 128.5 mm
- net Net-(R24-Pad2): track 4.98 -> 52.8 mm
- net Net-(R22-Pad2): track 4.53 -> 46.6 mm
- net /ACC_DRDY: track 27.7 -> 69.7 mm
- net /PWM_A: track 25.2 -> 58.5 mm
- net VCC: track 184.1 -> 153.8 mm
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
Commit message: PCB v3
PCB v3
Parts:
- moved C36 4.59 mm to (128.8, 136.6), turned to 180 degrees
- moved ? 4.05 mm to (105.5, 171.3)
- moved C40 2.94 mm to (125.0, 137.3)
- moved C30 2.40 mm to (126.0, 122.7)
- moved C32 2.38 mm to (128.7, 122.7)
- moved C46 1.53 mm to (121.5, 136.5), turned to 180 degrees
- moved C15 0.45 mm to (100.5, 161.0)
- moved P3 0.45 mm to (114.2, 168.1)
- moved Y1 0.40 mm to (97.0, 157.2)
- moved C4 0.30 mm to (101.5, 152.2)
- moved C33 0.22 mm to (89.1, 126.4)
Routing:
- net GND: track 569.3 -> 641.6 mm
- net +3V3: track 413.4 -> 397.1 mm
- net /ACC_DRDY: track 69.7 -> 79.1 mm
- net /INT_10_2: track 38.0 -> 46.5 mm
- net VCC: track 153.8 -> 159.1 mm
- net +5V: track 246.3 -> 248.9 mm
- net /SHARP_3: track 89.5 -> 91.9 mm
- net /INT_10_1: track 49.0 -> 47.2 mm
- net /SHARP_1: track 89.9 -> 91.5 mm
- net /ACC_INT2: track 90.6 -> 89.1 mm
- net /SCL: track 128.5 -> 129.6 mm
- net /START: track 33.2 -> 32.4 mm
- net /MOSI: track 59.9 -> 60.7 mm
- net /SCK: track 51.8 -> 52.5 mm
- net /SHARP_2: track 84.7 -> 85.4 mm
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